Commit message: fixed rotation axes of the wheels

File: my_rb1_description/urdf/my_rb1_robot.urdf (robot description, URDF)
Before this commit: robot my_rb1_robot, 7 links, 6 joints
Joints:
- joint base_link_left_wheel: axis 0 1 0 -> 0 0 1
- joint base_link_right_wheel: axis 0 1 0 -> 0 0 1

Commit message: resubmission

File: my_rb1_description/urdf/my_rb1_robot.urdf (robot description, URDF)
Before this commit: robot my_rb1_robot, 7 links, 6 joints
Links:
- link back_caster: geometry collision sphere radius=0.025; visual sphere radius=0.025
- link front_caster: geometry collision sphere radius=0.025; visual sphere radius=0.025
- link left_wheel: geometry collision cylinder length=0.03 radius=0.025; visual cylinder length=0.03 radius=0.025
- link right_wheel: geometry collision cylinder length=0.03 radius=0.025; visual cylinder length=0.03 radius=0.025
Joints:
- removed joint base_link_back_caster
- removed joint base_link_base_footprint
- removed joint base_link_front_caster
- removed joint base_link_front_laser
- removed joint base_link_left_wheel
- removed joint base_link_right_wheel
- added joint base_link_back_caster_joint: type fixed, parent base_link, child back_caster, origin xyz=0.1 0.0 -0.15 rpy=0 0 0
- added joint base_link_front_caster_joint: type fixed, parent base_link, child front_caster, origin xyz=-0.1 0.0 -0.15 rpy=0 0 0
- added joint base_link_front_laser_joint: type fixed, parent base_link, child front_laser, origin xyz=0.25 0 0.075 rpy=3.14 0 0
- added joint base_link_left_wheel_joint: type continuous, parent base_link, child left_wheel, origin xyz=0 -0.2 -0.15 rpy=0 0 0, axis 0 1 0
- added joint base_link_plate_joint: type fixed, parent base_footprint, child base_link, origin xyz=0 0 0.15 rpy=0 0 0
- added joint base_link_right_wheel_joint: type continuous, parent base_link, child right_wheel, origin xyz=0 0.2 -0.15 rpy=0 0 0, axis 0 1 0
